Commit message: barista xacro fix

File: urdf/barista.xacro (robot description, xacro)
@@ -2,7 +2,7 @@
 <robot name="BaristaII"
   xmlns:xacro="http://www.ros.org/wiki/xacro">
-  <xacro:include filename="$(find barista_bot)/urdf/materials.xacro" />
-  <xacro:include filename="$(find barista_bot)/urdf/barista.gazebo" />
-  <xacro:include filename="$(find barista_bot)/urdf/macros.xacro" />
+  <xacro:include filename="$(find waiter_robot)/urdf/materials.xacro" />
+  <xacro:include filename="$(find waiter_robot)/urdf/barista.gazebo" />
+  <xacro:include filename="$(find waiter_robot)/urdf/macros.xacro" />
   <xacro:property name="casterRadius" value="0.049"/>
   <xacro:property name="casterMass" value="1"/>
@@ -265,5 +265,5 @@
       <origin rpy="0 0 0" xyz="0 0 0"/>
       <geometry>
-        <mesh filename="package://barista_bot/meshes/hokuyo.dae" />
+        <mesh filename="package://waiter_robot/meshes/hokuyo.dae" />
       </geometry>
     </visual>
